File: Atmel ATmega 328P PLC OUTPUTS.sch (KiCad schematic (older format))
At the start: 32 parts, among them J12 Screw_Terminal_01x02, J13 Screw_Terminal_01x02, J14 Screw_Terminal_01x03, J15 Screw_Terminal_01x03, J16 Screw_Terminal_01x03, U10 PC817, U11 PC817, U12 PC817, U13 PC817, U14 PC817, U8 LM7810_TO220, U9 LM7810_TO220

Commit message: Finished schematic with all elements.
Parts:
- C14, C15: value C -> 1uF 16V
- D10, D11, D12: value LED -> GREEN
- D13, D14, D15: value D -> LS4148
- R27, R28, R33, R34, R35: value R -> 10k
- R29, R30: value R -> 1k
- R31, R32: value R -> 680R
Connections:
- net +24V: now also U8.1 (VI), U9.1 (VI)
- net +5V: now also D13.1 (K), D14.1 (K), D15.1 (K), RLY1.2 (COIL), RLY2.2 (COIL), RLY3.2 (COIL)
- net GND: now also C14.2, C15.2, J12.2 (Pin_2), J13.2 (Pin_2), U10.2, U10.3, U11.2, U11.3, U12.2, U12.3, U13.2, U13.3, U14.2, U14.3, U8.2 (GND), U9.2 (GND)
- net PB1: now also R33.2
- net PB2: now also R34.2
- net PB3: now also R35.2
- net PD5: now also R27.2
- net PD6: now also R28.2
- net at U8.3 (VO): now also R29.2
- net at U10.1: now also R27.1
- net at U10.4: now also R29.1, R31.1
- net at R31.2: now also C14.1, J12.1 (Pin_1)
- net at U9.3 (VO): now also R30.2
- net at U11.1: now also R28.1
- net at U11.4: now also R30.1, R32.1
- net at R32.2: now also C15.1, J13.1 (Pin_1)
- net at R33.1: now also D10.2 (A)
- net at D10.1 (K): now also U12.1
- net at U12.4: now also D13.2 (A), RLY1.5 (COIL)
- net at RLY1.1 (COM): now also J14.2 (Pin_2)
- net at RLY1.3 (NO): now also J14.3 (Pin_3)
- net at RLY1.4 (NC): now also J14.1 (Pin_1)
- net at R34.1: now also D11.2 (A)
- net at D11.1 (K): now also U13.1
- net at U13.4: now also D14.2 (A), RLY2.5 (COIL)
- net at RLY2.1 (COM): now also J15.2 (Pin_2)
- net at RLY2.3 (NO): now also J15.3 (Pin_3)
- net at RLY2.4 (NC): now also J15.1 (Pin_1)
- net at R35.1: now also D12.2 (A)
- net at D12.1 (K): now also U14.1
- net at U14.4: now also D15.2 (A), RLY3.5 (COIL)
- net at RLY3.1 (COM): now also J16.2 (Pin_2)
- net at RLY3.3 (NO): now also J16.3 (Pin_3)
- net at RLY3.4 (NC): now also J16.1 (Pin_1)
Other:
- note added: "0 - 10V outputs (PWM)"
- note added: "10A Relay outputs"
- moved on the sheet: D10, D13, J12, J14, R33, RLY1, U12
